File: Connectors.kicad_sch (KiCad schematic)
At the start: 9 parts

Commit message: update traces
Parts:
- CP0: footprint (none) -> Apple-II:POWER; DigiKey (none) -> A14226-ND
- SLOT0: footprint (none) -> Apple-II:Standard_Edge_Connector; DigiKey (none) -> A31718-ND
- SLOT1, SLOT2, SLOT3, SLOT4, SLOT5, SLOT6, SLOT7: footprint (none) -> Apple-II:Standard_Edge_Connector
Connections:
- net GND: now also SLOT4.26 (Pin_26)
- net NC1: now reaches SLOT0.19 (Pin_19)
- net NC1: now also SLOT1.19 (Pin_19), SLOT2.19 (Pin_19), SLOT3.19 (Pin_19), SLOT4.19 (Pin_19), SLOT5.19 (Pin_19), SLOT6.19 (Pin_19), SLOT7.19 (Pin_19)
- net NC2: now reaches SLOT0.35 (Pin_35)
- net NC2: now also SLOT1.35 (Pin_35), SLOT2.35 (Pin_35), SLOT3.35 (Pin_35), SLOT4.35 (Pin_35), SLOT5.35 (Pin_35), SLOT6.35 (Pin_35), SLOT7.35 (Pin_35)
- no-connect marks 21 -> 4
