File: IO_AddressDecode.kicad_sch (KiCad schematic)
At the start: 39 parts, among them J0 Cassette Data In, J13 74LS74, J14 GAME_IO_Conn, J2 Cassette Data Out, K13 MA741, Q4 MPSA13

Commit message: update traces
Parts:
- removed J0: Cassette Data In, symbol AppleII-rescue:AudioJack2-Connector
- removed J2: Cassette Data Out, symbol AppleII-rescue:AudioJack2-Connector
- added J0: Cassette Data In, Connector_Audio:Jack_3.5mm_CUI_SJ1-3533NG_Horizontal_CircularHoles, symbol Connector_Audio:AudioJack2_Ground
- added J2: Cassette Data Out, Connector_Audio:Jack_3.5mm_CUI_SJ1-3533NG_Horizontal_CircularHoles, symbol Connector_Audio:AudioJack2_Ground
- A7: renamed from A1; footprint Apple:DIP-16_W7.62mm -> Package_DIP:DIP-16_W7.62mm_Socket_LongPads
- B10, H1, J13: footprint Apple:DIP-14_W7.62mm -> Package_DIP:DIP-14_W7.62mm
- CR1: footprint (none) -> Diode_THT:D_DO-15_P10.16mm_Horizontal
- Cap10, Cap11, Cap12, Cap5, Cap6, Cap7, Cap9: footprint (none) -> Capacitor_THT:C_Disc_D5.0mm_W2.5mm_P5.00mm
- Cap8: footprint (none) -> Capacitor_THT:C_Disc_D4.3mm_W1.9mm_P5.00mm
- F12: renamed from F3; footprint Apple:DIP-16_W7.62mm -> Package_DIP:DIP-16_W7.62mm
- F13, F14, H12, H13, H14, H2: footprint Apple:DIP-16_W7.62mm -> Package_DIP:DIP-16_W7.62mm
- J14: footprint Apple:DIP-16_W7.62mm -> Package_DIP:DIP-16_W7.62mm_Socket_LongPads
- JP-User1: footprint (none) -> Connector_PinSocket_2.54mm:PinSocket_1x02_P2.54mm_Vertical; now not fitted
- K13: footprint Apple:DIP-8_W7.62mm -> Package_DIP:DIP-8_W7.62mm
- Q4: footprint (none) -> Package_TO_SOT_THT:TO-92; Alt (none) -> KSP13; DigiKey (none) -> KSP13BU-ND
- SPKR1: footprint digikey-footprints:PinHeader_1x2_P2.54mm_Drill1.02mm -> Connector_PinSocket_2.54mm:PinSocket_1x02_P2.54mm_Vertical
Connections:
- net GND: now also J0.S, J2.S
- net at R18.2, R19.1: now also J2.T
- net at Cap10.1: now also J0.T
- no-connect marks 5 -> 7

Commit message: more tracing
Parts:
- J0, J2: footprint Connector_Audio:Jack_3.5mm_CUI_SJ1-3533NG_Horizontal_CircularHoles -> Apple-II:AUDIO_mono; DigiKey (none) -> CP-3502N-ND
Connections:
- net ROM_Select_D0 renamed ROM_SELECT_D0
- net ROM_Select_D8 renamed ROM_SELECT_D8
- net ROM_Select_E0 renamed ROM_SELECT_E0
- net ROM_Select_E8 renamed ROM_SELECT_E8
- net ROM_Select_F0 renamed ROM_SELECT_F0
- net ROM_Select_F8 renamed ROM_SELECT_F8
- net ~{IO-Select-1} renamed ~{IO-SELECT-1}
- net ~{IO-Select-2} renamed ~{IO-SELECT-2}
- net ~{IO-Select-3} renamed ~{IO-SELECT-3}
- net ~{IO-Select-4} renamed ~{IO-SELECT-4}
- net ~{IO-Select-5} renamed ~{IO-SELECT-5}
- net ~{IO-Select-6} renamed ~{IO-SELECT-6}
- net ~{IO-Select-7} renamed ~{IO-SELECT-7}

Commit message: more traces and nicer text
Connections:
- net GND: now also H14.6 (~{Y})
- no-connect marks 7 -> 6
Changed lines of the file:
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@@
   (no_connect (at 360.68 231.14))
   (no_connect (at 316.23 241.3))
-  (no_connect (at 156.21 106.68))
   (no_connect (at 331.47 195.834))
   (no_connect (at 318.77 241.3))
@@
         )
       )
+    )
+  )
+  (symbol (lib_id "power:GND") (at 156.21 106.68 270) (unit 1)
+    (in_bom yes) (on_board yes) (dnp no)
+    (property "Reference" "#PWR012" (at 149.86 106.68 0)
+      (effects (font (size 1.27 1.27)) hide)
+    )
+    (property "Value" "GND" (at 153.416 104.14 0)
+      (effects (font (size 1.27 1.27)))
+    )
+    (property "Footprint" "" (at 156.21 106.68 0)
+      (effects (font (size 1.27 1.27)) hide)
+    )
+    (property "Datasheet" "" (at 156.21 106.68 0)
+      (effects (font (size 1.27 1.27)) hide)
+    )
+    (pin "1")
+    (instances
+      (project "AppleII"
+        (path "/f1f08369-4db3-46f7-9b89-a5d3cfbed55a/00000000-0000-0000-0000-00006017a131"
+          (reference "#PWR012") (unit 1)
+        )
+      )

Commit message: more tracing
Connections:
- net Soft5 renamed SOFT5
Changed lines of the file:
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@@
     )
   )
-  (global_label "Soft5" (shape input) (at 302.26 186.69 180)
+  (global_label "SOFT5" (shape input) (at 302.26 186.69 180)
     (effects (font (size 1.27 1.27)) (justify right))
     (property "Intersheetrefs" "${INTERSHEET_REFS}" (at 302.26 186.69 0)
@@
     )
   )
-  (global_label "Soft5" (shape input) (at 316.23 50.8 180)
+  (global_label "SOFT5" (shape input) (at 316.23 50.8 180)
     (effects (font (size 1.27 1.27)) (justify right))
     (property "Intersheetrefs" "${INTERSHEET_REFS}" (at 316.23 50.8 0)

Commit message: more tracing - down to row E
Parts:
- added Cap1 (x3): 0.1uF, Capacitor_THT:C_Disc_D5.0mm_W2.5mm_P5.00mm, symbol Device:C_Small
Connections:
- net +5V: now also Cap1.2, Cap1.2, Cap1.2
- net GND: now also Cap1.1, Cap1.1, Cap1.1
- net SOFT5: now also B10.10 (~{S})
- no-connect marks 6 -> 7
Changed lines of the file:
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@@
   (junction (at 365.76 176.784) (diameter 0) (color 0 0 0 0)
   )
+  (junction (at 331.47 21.59) (diameter 0) (color 0 0 0 0)
+  )
   (junction (at 320.294 88.646) (diameter 0) (color 0 0 0 0)
   )
@@
   (junction (at 328.93 231.14) (diameter 0) (color 0 0 0 0)
   )
+  (junction (at 63.5 162.56) (diameter 0) (color 0 0 0 0)
+  )
   (junction (at 353.06 200.914) (diameter 0) (color 0 0 0 0)
   )
+  (junction (at 168.91 118.11) (diameter 0) (color 0 0 0 0)
+  )
   (no_connect (at 255.27 203.2))
   (no_connect (at 368.3 195.834))
   (no_connect (at 360.68 231.14))
+  (no_connect (at 240.03 198.12))
   (no_connect (at 316.23 241.3))
   (no_connect (at 331.47 195.834))
@@
     (stroke (width 0) (type default))
   )
+  (wire (pts (xy 59.69 162.56) (xy 63.5 162.56))
+    (stroke (width 0) (type default))
+  )
   (wire (pts (xy 328.93 223.52) (xy 328.93 231.14))
     (stroke (width 0) (type default))
@@
     (stroke (width 0) (type default))
   )
+  (wire (pts (xy 327.66 21.59) (xy 331.47 21.59))
+    (stroke (width 0) (type default))
+  )
   (wire (pts (xy 273.304 175.26) (xy 261.62 175.26))
     (stroke (width 0) (type default))
@@
     (stroke (width 0) (type default))
   )
-  (wire (pts (xy 331.47 21.336) (xy 331.47 22.86))
+  (wire (pts (xy 331.47 21.336) (xy 331.47 21.59))
     (stroke (width 0) (type default))
   )
@@
     (stroke (width 0) (type default))
   )
+  (wire (pts (xy 331.47 21.59) (xy 331.47 22.86))
+    (stroke (width 0) (type default))
+  )
   (wire (pts (xy 336.55 172.72) (xy 331.47 172.72))
     (stroke (width 0) (type default))
@@
     )
   )
+  (global_label "SOFT5" (shape input) (at 247.65 193.04 90) (fields_autoplaced)
+    (effects (font (size 1.27 1.27)) (justify left))
+    (property "Intersheetrefs" "${INTERSHEET_REFS}" (at 247.65 184.9033 90)
+      (effects (font (size 1.27 1.27)) (justify left) hide)
+    )
+  )
   (global_label "ROM_SELECT_F8" (shape output) (at 90.424 77.47 0) (fields_autoplaced)
     (effects (font (size 1.27 1.27)) (justify left))
@@
     )
   )
+  (symbol (lib_id "Device:C_Small") (at 325.12 21.59 90) (unit 1)
+    (in_bom yes) (on_board yes) (dnp no)
+    (property "Reference" "Cap1" (at 323.342 21.336 0)
+      (effects (font (size 1.27 1.27)) (justify left))
+    )
+    (property "Value" "0.1uF" (at 325.12 19.812 0)
+      (effects (font (size 1.27 1.27)) (justify left))
+    )
+    (property "Footprint" "Capacitor_THT:C_Disc_D5.0mm_W2.5mm_P5.00mm" (at 325.12 21.59 0)
+      (effects (font (size 1.27 1.27)) hide)
+    )
+    (property "Datasheet" "~" (at 325.12 21.59 0)
+      (effects (font (size 1.27 1.27)) hide)
+    )
+    (pin "1")
+    (pin "2")
+    (instances
+      (project "AppleII"
+        (path "/f1f08369-4db3-46f7-9b89-a5d3cfbed55a/00000000-0000-0000-0000-00006016cde0"
+          (reference "Cap1") (unit 1)
+        )
+        (path "/f1f08369-4db3-46f7-9b89-a5d3cfbed55a/00000000-0000-0000-0000-00006039aab4"
+          (reference "Cap3") (unit 1)
+        )
+        (path "/f1f08369-4db3-46f7-9b89-a5d3cfbed55a/00000000-0000-0000-0000-00006017a131"
+          (reference "Cap16") (unit 1)
+        )
+      )
+    )
+  )
   (symbol (lib_id "power:+5V") (at 237.998 162.56 0) (unit 1)
     (in_bom yes) (on_board yes) (dnp no)
@@
     )
   )
+  (symbol (lib_id "power:GND") (at 322.58 21.59 270) (unit 1)
+    (in_bom yes) (on_board yes) (dnp no)
+    (property "Reference" "#PWR013" (at 316.23 21.59 0)
+      (effects (font (size 1.27 1.27)) hide)
+    )
+    (property "Value" "GND" (at 318.1858 21.717 0)
+      (effects (font (size 1.27 1.27)))
+    )
+    (property "Footprint" "" (at 322.58 21.59 0)
+      (effects (font (size 1.27 1.27)) hide)
+    )
+    (property "Datasheet" "" (at 322.58 21.59 0)
+      (effects (font (size 1.27 1.27)) hide)
+    )
+    (pin "1")
+    (instances
+      (project "AppleII"
+        (path "/f1f08369-4db3-46f7-9b89-a5d3cfbed55a/00000000-0000-0000-0000-00006039aab4"
+          (reference "#PWR013") (unit 1)
+        )
+        (path "/f1f08369-4db3-46f7-9b89-a5d3cfbed55a/00000000-0000-0000-0000-00006017a131"
+          (reference "#PWR015") (unit 1)
+        )
+      )
+    )
+  )
   (symbol (lib_id "power:+5V") (at 63.5 51.054 0) (unit 1)
     (in_bom yes) (on_board yes) (dnp no)
@@
     )
   )
+  (symbol (lib_id "power:GND") (at 168.91 123.19 0) (unit 1)
+    (in_bom yes) (on_board yes) (dnp no)
+    (property "Reference" "#PWR013" (at 168.91 129.54 0)
+      (effects (font (size 1.27 1.27)) hide)
+    )
+    (property "Value" "GND" (at 169.037 127.5842 0)
+      (effects (font (size 1.27 1.27)))
+    )
+    (property "Footprint" "" (at 168.91 123.19 0)
+      (effects (font (size 1.27 1.27)) hide)
+    )
+    (property "Datasheet" "" (at 168.91 123.19 0)
+      (effects (font (size 1.27 1.27)) hide)
+    )
+    (pin "1")
+    (instances
+      (project "AppleII"
+        (path "/f1f08369-4db3-46f7-9b89-a5d3cfbed55a/00000000-0000-0000-0000-00006039aab4"
+          (reference "#PWR013") (unit 1)
+        )
+        (path "/f1f08369-4db3-46f7-9b89-a5d3cfbed55a/00000000-0000-0000-0000-00006017a131"
+          (reference "#PWR018") (unit 1)
+        )
+      )
+    )
+  )
+  (symbol (lib_id "Device:C_Small") (at 168.91 120.65 180) (unit 1)
+    (in_bom yes) (on_board yes) (dnp no)
+    (property "Reference" "Cap1" (at 168.656 122.428 0)
+      (effects (font (size 1.27 1.27)) (justify left))
+    )
+    (property "Value" "0.1uF" (at 167.132 120.65 0)
+      (effects (font (size 1.27 1.27)) (justify left))
+    )
+    (property "Footprint" "Capacitor_THT:C_Disc_D5.0mm_W2.5mm_P5.00mm" (at 168.91 120.65 0)
+      (effects (font (size 1.27 1.27)) hide)
+    )
+    (property "Datasheet" "~" (at 168.91 120.65 0)
+      (effects (font (size 1.27 1.27)) hide)
+    )
+    (pin "1")
+    (pin "2")
+    (instances
+      (project "AppleII"
+        (path "/f1f08369-4db3-46f7-9b89-a5d3cfbed55a/00000000-0000-0000-0000-00006016cde0"
+          (reference "Cap1") (unit 1)
+        )
+        (path "/f1f08369-4db3-46f7-9b89-a5d3cfbed55a/00000000-0000-0000-0000-00006039aab4"
+          (reference "Cap3") (unit 1)
+        )
+        (path "/f1f08369-4db3-46f7-9b89-a5d3cfbed55a/00000000-0000-0000-0000-00006017a131"
+          (reference "Cap19") (unit 1)
+        )
+      )
+    )
+  )
   (symbol (lib_id "power:GND") (at 237.998 181.356 0) (unit 1)
     (in_bom yes) (on_board yes) (dnp no)
@@
     )
   )
+  (symbol (lib_id "Device:C_Small") (at 57.15 162.56 90) (unit 1)
+    (in_bom yes) (on_board yes) (dnp no)
+    (property "Reference" "Cap1" (at 55.372 162.306 0)
+      (effects (font (size 1.27 1.27)) (justify left))
+    )
+    (property "Value" "0.1uF" (at 57.15 160.782 0)
+      (effects (font (size 1.27 1.27)) (justify left))
+    )
+    (property "Footprint" "Capacitor_THT:C_Disc_D5.0mm_W2.5mm_P5.00mm" (at 57.15 162.56 0)
+      (effects (font (size 1.27 1.27)) hide)
+    )
+    (property "Datasheet" "~" (at 57.15 162.56 0)
+      (effects (font (size 1.27 1.27)) hide)
+    )
+    (pin "1")
+    (pin "2")
+    (instances
+      (project "AppleII"
+        (path "/f1f08369-4db3-46f7-9b89-a5d3cfbed55a/00000000-0000-0000-0000-00006016cde0"
+          (reference "Cap1") (unit 1)
+        )
+        (path "/f1f08369-4db3-46f7-9b89-a5d3cfbed55a/00000000-0000-0000-0000-00006039aab4"
+          (reference "Cap3") (unit 1)
+        )
+        (path "/f1f08369-4db3-46f7-9b89-a5d3cfbed55a/00000000-0000-0000-0000-00006017a131"
+          (reference "Cap18") (unit 1)
+        )
+      )
+    )
+  )
   (symbol (lib_id "power:-12V") (at 263.652 164.592 0) (unit 1)
     (in_bom yes) (on_board yes) (dnp no)
@@
         )
       )
+    )
+  )
+  (symbol (lib_id "power:GND") (at 54.61 162.56 270) (unit 1)
+    (in_bom yes) (on_board yes) (dnp no)
+    (property "Reference" "#PWR013" (at 48.26 162.56 0)
+      (effects (font (size 1.27 1.27)) hide)
+    )
+    (property "Value" "GND" (at 50.2158 162.687 0)
+      (effects (font (size 1.27 1.27)))
+    )
+    (property "Footprint" "" (at 54.61 162.56 0)
+      (effects (font (size 1.27 1.27)) hide)
+    )
+    (property "Datasheet" "" (at 54.61 162.56 0)
+      (effects (font (size 1.27 1.27)) hide)
+    )
+    (pin "1")
+    (instances
+      (project "AppleII"
+        (path "/f1f08369-4db3-46f7-9b89-a5d3cfbed55a/00000000-0000-0000-0000-00006039aab4"
+          (reference "#PWR013") (unit 1)
+        )
+        (path "/f1f08369-4db3-46f7-9b89-a5d3cfbed55a/00000000-0000-0000-0000-00006017a131"
+          (reference "#PWR017") (unit 1)
+        )
+      )

Commit message: more tracing
Parts:
- renumbered Cap1 to Cap16, Cap1 to Cap18, Cap1 to Cap19
Changed lines of the file:
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@@
   (symbol (lib_id "Device:C_Small") (at 325.12 21.59 90) (unit 1)
     (in_bom yes) (on_board yes) (dnp no)
-    (property "Reference" "Cap1" (at 323.342 21.336 0)
+    (property "Reference" "Cap16" (at 323.342 21.336 0)
       (effects (font (size 1.27 1.27)) (justify left))
     )
@@
     (instances
       (project "AppleII"
-        (path "/f1f08369-4db3-46f7-9b89-a5d3cfbed55a/00000000-0000-0000-0000-00006016cde0"
-          (reference "Cap1") (unit 1)
-        )
-        (path "/f1f08369-4db3-46f7-9b89-a5d3cfbed55a/00000000-0000-0000-0000-00006039aab4"
-          (reference "Cap3") (unit 1)
-        )
         (path "/f1f08369-4db3-46f7-9b89-a5d3cfbed55a/00000000-0000-0000-0000-00006017a131"
           (reference "Cap16") (unit 1)
@@
   (symbol (lib_id "power:GND") (at 322.58 21.59 270) (unit 1)
     (in_bom yes) (on_board yes) (dnp no)
-    (property "Reference" "#PWR013" (at 316.23 21.59 0)
+    (property "Reference" "#PWR015" (at 316.23 21.59 0)
       (effects (font (size 1.27 1.27)) hide)
     )
@@
     (instances
       (project "AppleII"
-        (path "/f1f08369-4db3-46f7-9b89-a5d3cfbed55a/00000000-0000-0000-0000-00006039aab4"
-          (reference "#PWR013") (unit 1)
-        )
         (path "/f1f08369-4db3-46f7-9b89-a5d3cfbed55a/00000000-0000-0000-0000-00006017a131"
           (reference "#PWR015") (unit 1)
@@
   (symbol (lib_id "power:GND") (at 168.91 123.19 0) (unit 1)
     (in_bom yes) (on_board yes) (dnp no)
-    (property "Reference" "#PWR013" (at 168.91 129.54 0)
+    (property "Reference" "#PWR018" (at 168.91 129.54 0)
       (effects (font (size 1.27 1.27)) hide)
     )
@@
     (instances
       (project "AppleII"
-        (path "/f1f08369-4db3-46f7-9b89-a5d3cfbed55a/00000000-0000-0000-0000-00006039aab4"
-          (reference "#PWR013") (unit 1)
-        )
         (path "/f1f08369-4db3-46f7-9b89-a5d3cfbed55a/00000000-0000-0000-0000-00006017a131"
           (reference "#PWR018") (unit 1)
@@
   (symbol (lib_id "Device:C_Small") (at 168.91 120.65 180) (unit 1)
     (in_bom yes) (on_board yes) (dnp no)
-    (property "Reference" "Cap1" (at 168.656 122.428 0)
+    (property "Reference" "Cap19" (at 168.656 122.428 0)
       (effects (font (size 1.27 1.27)) (justify left))
     )
@@
     (instances
       (project "AppleII"
-        (path "/f1f08369-4db3-46f7-9b89-a5d3cfbed55a/00000000-0000-0000-0000-00006016cde0"
-          (reference "Cap1") (unit 1)
-        )
-        (path "/f1f08369-4db3-46f7-9b89-a5d3cfbed55a/00000000-0000-0000-0000-00006039aab4"
-          (reference "Cap3") (unit 1)
-        )
         (path "/f1f08369-4db3-46f7-9b89-a5d3cfbed55a/00000000-0000-0000-0000-00006017a131"
           (reference "Cap19") (unit 1)
@@
   (symbol (lib_id "Device:C_Small") (at 57.15 162.56 90) (unit 1)
     (in_bom yes) (on_board yes) (dnp no)
-    (property "Reference" "Cap1" (at 55.372 162.306 0)
+    (property "Reference" "Cap18" (at 55.372 162.306 0)
       (effects (font (size 1.27 1.27)) (justify left))
     )
@@
     (instances
       (project "AppleII"
-        (path "/f1f08369-4db3-46f7-9b89-a5d3cfbed55a/00000000-0000-0000-0000-00006016cde0"
-          (reference "Cap1") (unit 1)
-        )
-        (path "/f1f08369-4db3-46f7-9b89-a5d3cfbed55a/00000000-0000-0000-0000-00006039aab4"
-          (reference "Cap3") (unit 1)
-        )
         (path "/f1f08369-4db3-46f7-9b89-a5d3cfbed55a/00000000-0000-0000-0000-00006017a131"
           (reference "Cap18") (unit 1)
@@
   (symbol (lib_id "power:GND") (at 54.61 162.56 270) (unit 1)
     (in_bom yes) (on_board yes) (dnp no)
-    (property "Reference" "#PWR013" (at 48.26 162.56 0)
+    (property "Reference" "#PWR017" (at 48.26 162.56 0)
       (effects (font (size 1.27 1.27)) hide)
     )
@@
     (instances
       (project "AppleII"
-        (path "/f1f08369-4db3-46f7-9b89-a5d3cfbed55a/00000000-0000-0000-0000-00006039aab4"
-          (reference "#PWR013") (unit 1)
-        )
         (path "/f1f08369-4db3-46f7-9b89-a5d3cfbed55a/00000000-0000-0000-0000-00006017a131"
           (reference "#PWR017") (unit 1)

Commit message: finish tracing
Parts:
- added J3: Conn_01x16, Connector_PinHeader_2.54mm:PinHeader_1x16_P2.54mm_Vertical, symbol Connector_Generic:Conn_01x16
Connections:
- net +5V: now also J3.2 (Pin_2)
- net -12V: now also J3.3 (Pin_3)
- net GND: now also J3.7 (Pin_7)
- net KBD_Data0: now also J3.4 (Pin_4)
- net KBD_Data1: now also J3.1 (Pin_1)
- net KBD_Data2: now also J3.6 (Pin_6)
- net KBD_Data3: now also J3.5 (Pin_5)
- net KBD_Data4: now also J3.11 (Pin_11)
- net KBD_Data5: now also J3.10 (Pin_10)
- net KBD_Data6: now also J3.12 (Pin_12)
- net ~{RESET}: now also J3.9 (Pin_9)
- net at A7.2 (STROBE), B10.11 (C): now also J3.8 (Pin_8)
- no-connect marks 7 -> 11
