File: ClockGen.kicad_sch (KiCad schematic)
At the start: 21 parts, among them Q1 2N4258, Q2 2N4258, Y1 XT0001

Commit message: update traces
Parts:
- A2, B12, B13, B2, C11, D2: footprint Apple:DIP-14_W7.62mm -> Package_DIP:DIP-14_W7.62mm
- B1, C1, C2, D11, D12, D13, D14: footprint Apple:DIP-16_W7.62mm -> Package_DIP:DIP-16_W7.62mm
- Cap1: footprint (none) -> Capacitor_THT:C_Disc_D5.0mm_W2.5mm_P5.00mm
- Q1, Q2: footprint (none) -> Package_TO_SOT_THT:TO-18-3; Alt (none) -> 2N4208; DigiKey (none) -> 2N4208-ND
- Y1: footprint (none) -> Crystal:Crystal_HC18-U_Vertical
Changed lines of the file:
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@@
       (effects (font (size 1.27 1.27)))
     )
-    (property "Footprint" "Apple:DIP-16_W7.62mm" (at 152.4 77.47 0)
+    (property "Footprint" "Package_DIP:DIP-16_W7.62mm" (at 152.4 77.47 0)
       (effects (font (size 1.27 1.27)) hide)
     )
@@
       (effects (font (size 1.27 1.27)) (justify left))
     )
-    (property "Footprint" "" (at 35.56 43.18 0)
+    (property "Footprint" "Package_TO_SOT_THT:TO-18-3" (at 35.56 43.18 0)
       (effects (font (size 1.27 1.27)) hide)
     )
@@
       (effects (font (size 1.27 1.27)) hide)
     )
+    (property "Alt" "2N4208" (at 40.64 40.64 0)
+      (effects (font (size 1.27 1.27)) hide)
+    )
+    (property "DigiKey" "2N4208-ND" (at 40.64 40.64 0)
+      (effects (font (size 1.27 1.27)) hide)
+    )
     (pin "1")
     (pin "2")
@@
       (effects (font (size 1.27 1.27)) (justify left))
     )
-    (property "Footprint" "" (at 27.94 43.18 0)
+    (property "Footprint" "Package_TO_SOT_THT:TO-18-3" (at 27.94 43.18 0)
       (effects (font (size 1.27 1.27)) hide)
     )
@@
       (effects (font (size 1.27 1.27)) hide)
     )
+    (property "Alt" "2N4208" (at 22.86 40.64 0)
+      (effects (font (size 1.27 1.27)) hide)
+    )
+    (property "DigiKey" "2N4208-ND" (at 22.86 40.64 0)
+      (effects (font (size 1.27 1.27)) hide)
+    )
     (pin "1")
     (pin "2")
@@
       (effects (font (size 1.27 1.27)))
     )
-    (property "Footprint" "Apple:DIP-16_W7.62mm" (at 152.4 123.19 0)
+    (property "Footprint" "Package_DIP:DIP-16_W7.62mm" (at 152.4 123.19 0)
       (effects (font (size 1.27 1.27)) hide)
     )
@@
       (effects (font (size 1.27 1.27)) (justify left))
     )
-    (property "Footprint" "" (at 56.642 45.72 0)
+    (property "Footprint" "Capacitor_THT:C_Disc_D5.0mm_W2.5mm_P5.00mm" (at 56.642 45.72 0)
       (effects (font (size 1.27 1.27)) hide)
     )
@@
       (effects (font (size 1.27 1.27)))
     )
-    (property "Footprint" "" (at 31.75 50.8 0)
+    (property "Footprint" "Crystal:Crystal_HC18-U_Vertical" (at 31.75 50.8 0)
       (effects (font (size 1.27 1.27)) hide)
     )
@@
       (effects (font (size 1.27 1.27)))
     )
-    (property "Footprint" "Apple:DIP-16_W7.62mm" (at 152.4 166.37 0)
+    (property "Footprint" "Package_DIP:DIP-16_W7.62mm" (at 152.4 166.37 0)
       (effects (font (size 1.27 1.27)) hide)
     )
@@
       (effects (font (size 1.27 1.27)))
     )
-    (property "Footprint" "Apple:DIP-16_W7.62mm" (at 152.4 212.09 0)
+    (property "Footprint" "Package_DIP:DIP-16_W7.62mm" (at 152.4 212.09 0)
       (effects (font (size 1.27 1.27)) hide)
     )
@@
       (effects (font (size 1.27 1.27)) (justify left))
     )
-    (property "Footprint" "Apple:DIP-14_W7.62mm" (at 140.97 54.61 0)
+    (property "Footprint" "Package_DIP:DIP-14_W7.62mm" (at 140.97 54.61 0)
       (effects (font (size 1.27 1.27)) hide)
     )
@@
       (effects (font (size 1.27 1.27)))
     )
-    (property "Footprint" "Apple:DIP-16_W7.62mm" (at 230.378 180.594 0)
+    (property "Footprint" "Package_DIP:DIP-16_W7.62mm" (at 230.378 180.594 0)
       (effects (font (size 1.27 1.27)) hide)
     )
@@
       (effects (font (size 1.27 1.27)))
     )
-    (property "Footprint" "Apple:DIP-16_W7.62mm" (at 281.178 172.974 0)
+    (property "Footprint" "Package_DIP:DIP-16_W7.62mm" (at 281.178 172.974 0)
       (effects (font (size 1.27 1.27)) hide)
     )
@@
       (effects (font (size 1.27 1.27)))
     )
-    (property "Footprint" "Apple:DIP-14_W7.62mm" (at 72.39 50.8 0)
+    (property "Footprint" "Package_DIP:DIP-14_W7.62mm" (at 72.39 50.8 0)
       (effects (font (size 1.27 1.27)) hide)
     )
@@
       (effects (font (size 1.27 1.27)))
     )
-    (property "Footprint" "Apple:DIP-14_W7.62mm" (at 229.616 88.9 0)
+    (property "Footprint" "Package_DIP:DIP-14_W7.62mm" (at 229.616 88.9 0)
       (effects (font (size 1.27 1.27)) hide)
     )
@@
       (effects (font (size 1.27 1.27)))
     )
-    (property "Footprint" "Apple:DIP-14_W7.62mm" (at 191.008 165.1 0)
+    (property "Footprint" "Package_DIP:DIP-14_W7.62mm" (at 191.008 165.1 0)
       (effects (font (size 1.27 1.27)) hide)
     )
@@
       (effects (font (size 1.27 1.27)))
     )
-    (property "Footprint" "Apple:DIP-14_W7.62mm" (at 197.104 137.668 0)
+    (property "Footprint" "Package_DIP:DIP-14_W7.62mm" (at 197.104 137.668 0)
       (effects (font (size 1.27 1.27)) hide)
     )
@@
       (effects (font (size 1.27 1.27)))
     )
-    (property "Footprint" "Apple:DIP-16_W7.62mm" (at 252.476 99.06 0)
+    (property "Footprint" "Package_DIP:DIP-16_W7.62mm" (at 252.476 99.06 0)
       (effects (font (size 1.27 1.27)) hide)
     )
@@
       (effects (font (size 1.27 1.27)))
     )
-    (property "Footprint" "Apple:DIP-14_W7.62mm" (at 188.214 185.42 0)
+    (property "Footprint" "Package_DIP:DIP-14_W7.62mm" (at 188.214 185.42 0)
       (effects (font (size 1.27 1.27)) hide)
     )
@@
       (effects (font (size 1.27 1.27)) (justify right))
     )
-    (property "Footprint" "Apple:DIP-14_W7.62mm" (at 246.38 154.94 0)
+    (property "Footprint" "Package_DIP:DIP-14_W7.62mm" (at 246.38 154.94 0)
       (effects (font (size 1.27 1.27)) hide)
     )
@@
       (effects (font (size 1.27 1.27)))
     )
-    (property "Footprint" "Apple:DIP-14_W7.62mm" (at 208.28 170.434 0)
-      (effects (font (size 1.27 1.27)) hide)
-    )
+    (property "Footprint" "Package_DIP:DIP-14_W7.62mm" (at 208.28 170.434 0)
+      (effects (font (size 1.27 1.27)) hide)
+    )

Commit message: more tracing
Connections:
- net at D12.10 (CET), D12.3 (D0), D12.5 (D2)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: no longer C11.8, D11.9 (~{PE}), D12.9 (~{PE})
- new net: C11.8, D11.9 (~{PE}), D12.9 (~{PE})
Changed lines of the file:
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@@
   (junction (at 137.16 115.57) (diameter 0) (color 0 0 0 0)
-  )
-  (junction (at 137.16 123.19) (diameter 0) (color 0 0 0 0)
   )
   (junction (at 137.16 69.85) (diameter 0) (color 0 0 0 0)
@@
     (stroke (width 0) (type default))
   )
-  (bus_entry (at 171.45 116.84) (size 2.54 -2.54)
-    (stroke (width 0) (type default))
-  )
   (bus_entry (at 167.64 210.82) (size 2.54 -2.54)
     (stroke (width 0) (type default))
@@
     (stroke (width 0) (type default))
   )
-  (bus_entry (at 171.45 165.1) (size 2.54 -2.54)
-    (stroke (width 0) (type default))
-  )
   (bus_entry (at 167.64 205.74) (size 2.54 -2.54)
     (stroke (width 0) (type default))
@@
     (stroke (width 0) (type default))
   )
-  (bus_entry (at 171.45 114.3) (size 2.54 -2.54)
-    (stroke (width 0) (type default))
-  )
   (bus_entry (at 168.91 68.58) (size -2.54 2.54)
     (stroke (width 0) (type default))
@@
     (stroke (width 0) (type default))
   )
-  (bus (pts (xy 173.99 107.95) (xy 184.15 107.95))
-    (stroke (width 0) (type default))
-  )
   (wire (pts (xy 250.19 167.894) (xy 243.078 167.894))
     (stroke (width 0) (type default))
@@
     (stroke (width 0) (type default))
   )
-  (wire (pts (xy 137.16 123.19) (xy 137.16 143.51))
-    (stroke (width 0) (type default))
-  )
   (wire (pts (xy 149.86 95.25) (xy 151.13 95.25))
     (stroke (width 0) (type default))
@@
     (stroke (width 0) (type default))
   )
-  (wire (pts (xy 132.08 123.19) (xy 137.16 123.19))
+  (wire (pts (xy 132.08 123.19) (xy 139.7 123.19))
     (stroke (width 0) (type default))
   )
@@
     (stroke (width 0) (type default))
   )
-  (wire (pts (xy 137.16 118.11) (xy 137.16 123.19))
+  (wire (pts (xy 137.16 118.11) (xy 137.16 143.51))
     (stroke (width 0) (type default))
   )
@@
     (stroke (width 0) (type default))
   )
-  (bus (pts (xy 173.99 107.95) (xy 173.99 111.76))
-    (stroke (width 0) (type default))
-  )
   (wire (pts (xy 163.83 73.66) (xy 166.37 73.66))
     (stroke (width 0) (type default))
@@
     (stroke (width 0) (type default))
   )
-  (bus (pts (xy 173.99 111.76) (xy 173.99 114.3))
-    (stroke (width 0) (type default))
-  )
   (wire (pts (xy 262.89 193.294) (xy 268.478 193.294))
     (stroke (width 0) (type default))
@@
     (stroke (width 0) (type default))
   )
-  (wire (pts (xy 137.16 123.19) (xy 139.7 123.19))
-    (stroke (width 0) (type default))
-  )
   (wire (pts (xy 163.83 133.35) (xy 167.64 133.35))
     (stroke (width 0) (type default))
@@
   )
   (bus (pts (xy 170.18 157.48) (xy 170.18 194.31))
-    (stroke (width 0) (type default))
-  )
-  (bus (pts (xy 173.99 114.3) (xy 173.99 162.56))
     (stroke (width 0) (type default))
   )
@@
     )
   )
+  (global_label "VC" (shape output) (at 171.45 116.84 0) (fields_autoplaced)
+    (effects (font (size 1.27 1.27)) (justify left))
+    (property "Intersheetrefs" "${INTERSHEET_REFS}" (at 176.1396 116.84 0)
+      (effects (font (size 1.27 1.27)) (justify left) hide)
+    )
+  )
   (global_label "~{7M}" (shape output) (at 267.97 106.68 0)
     (effects (font (size 1.27 1.27)) (justify left))
@@
     )
   )
+  (global_label "VA" (shape output) (at 171.45 165.1 0) (fields_autoplaced)
+    (effects (font (size 1.27 1.27)) (justify left))
+    (property "Intersheetrefs" "${INTERSHEET_REFS}" (at 175.9582 165.1 0)
+      (effects (font (size 1.27 1.27)) (justify left) hide)
+    )
+  )
   (global_label "~{RAS}" (shape output) (at 250.19 167.894 0)
     (effects (font (size 1.27 1.27)) (justify left))
@@
     )
   )
-  (global_label "V[A..C]" (shape output) (at 184.15 107.95 0)
-    (effects (font (size 1.27 1.27)) (justify left))
-    (property "Intersheetrefs" "${INTERSHEET_REFS}" (at 184.15 107.95 0)
-      (effects (font (size 1.27 1.27)) hide)
-    )
-  )
   (global_label "PHI0" (shape output) (at 267.97 93.98 0)
     (effects (font (size 1.27 1.27)) (justify left))
@@
     )
   )
+  (global_label "VB" (shape output) (at 171.45 114.3 0) (fields_autoplaced)
+    (effects (font (size 1.27 1.27)) (justify left))
+    (property "Intersheetrefs" "${INTERSHEET_REFS}" (at 176.1396 114.3 0)
+      (effects (font (size 1.27 1.27)) (justify left) hide)
+    )
+  )

Commit message: finish tracing
Parts:
- removed Q1, Q2: 2N4258, Package_TO_SOT_THT:TO-18-3, symbol Device:Q_PNP_BCE
- added unit 5 of A2
- added unit 5 of B13
- added unit 5 of B2
- added Cap29 (x2), Cap41 (x3): 0.1uF, Capacitor_THT:C_Disc_D5.0mm_W2.5mm_P5.00mm, symbol Device:C_Small
- added Q1, Q2: 2N4258, Package_TO_SOT_THT:TO-18-3, symbol Device:Q_PNP_EBC
Connections:
- net +5V: now also A2.14 (VCC), B13.14 (VCC), B2.14 (VCC), Cap29.2, Cap29.2, Cap41.2, Cap41.2, Cap41.2, Q1.2 (B)
- net GND: now also A2.7 (GND), B13.7 (GND), B2.7 (GND), Cap29.1, Cap29.1, Cap41.1, Cap41.1, Cap41.1
- net SOFT5: now also D11.1 (~{MR}), D12.1 (~{MR})
- net at R4.2, Y1.2: now also Q2.2 (B)
- net at B2.10, R3.1: now also Q2.3 (C)
- net at R1.2: now also Q1.1 (E), Q2.1 (E)
- net at R2.1, Y1.1: now also Q1.3 (C)
