File: RAMAddressMux.kicad_sch (KiCad schematic)
At the start: 22 parts, among them J1 74LS257

Commit message: add missing test points
Parts:
- added TP1: TestPoint, TestPoint:TestPoint_THTPad_1.5x1.5mm_Drill0.7mm, symbol Connector:TestPoint
Connections:
- net at D1.1, E1.1, E2.4 (O0): now also TP1.1
Other:
- moved on the sheet: C11A, C11C, C12, Cap44, Cap49, E11, E12, E13, E14, H1C, H1D, RA02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
