File: Video Gen.kicad_sch (KiCad schematic)
At the start: 37 parts, among them J18 Aux Video, K14 RCA Connector, Q3 2N3904

Commit message: add alternative char gen footprint
Parts:
- added Aalt5: 2513->2716, Package_DIP:DIP-24_W15.24mm_Socket, symbol Connector_Generic:Conn_02x12_Counter_Clockwise
- added D21, D22, D23: BAT54A, Package_TO_SOT_SMD:SOT-23, symbol Diode:BAT54A
Connections:
- net +5V: now also Aalt5.21 (Pin_21), Aalt5.24 (Pin_24)
- net GND: now also Aalt5.12 (Pin_12), Aalt5.18 (Pin_18), Aalt5.19 (Pin_19), Aalt5.20 (Pin_20), Aalt5.22 (Pin_22), D21.3, D22.3, D23.3
- net LD0: now also Aalt5.5 (Pin_5), D22.2
- net LD1: now also Aalt5.4 (Pin_4), D22.1
- net LD2: now also Aalt5.3 (Pin_3), D21.2
- net LD3: now also Aalt5.2 (Pin_2), D21.1
- net LD4: now also Aalt5.1 (Pin_1), D23.2
- net LD5: now also Aalt5.23 (Pin_23), D23.1
- net VA: now also Aalt5.8 (Pin_8)
- net VB: now also Aalt5.7 (Pin_7)
- net VC: now also Aalt5.6 (Pin_6)
- net O1: now reaches A3.4 (C), A5.4 (O1)
- net O1: now also Aalt5.9 (Pin_9)
- net O2: now reaches A3.5 (D), A5.5 (O2)
- net O2: now also Aalt5.10 (Pin_10)
- net O3: now reaches A3.10 (E), A5.6 (O3)
- net O3: now also Aalt5.11 (Pin_11)
- net O4: now reaches A3.11 (F), A5.7 (O4)
- net O4: now also Aalt5.13 (Pin_13)
- net O5: now reaches A3.12 (G), A5.8 (O5)
- net O5: now also Aalt5.14 (Pin_14)
- no-connect marks 8 -> 11
