File: AppleII.kicad_pcb (KiCad board)
At the start: 2 copper layers, 215.5 x 361.2 mm, 203 parts, among them J0 Cassette Data In, J1 74LS257, J13 74LS74, J14 GAME_IO_Conn, J18 Aux Video, J2 Cassette Data Out, J3 Conn_01x16, J4 Conn_01x25, J5 Conn_01x25, J6 Conn_01x24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

Commit message: fix assignment of LD0-7 net
Connections:
- net LD0 renamed /CPU Tranceiver Driver and Data MUX/LD0
- net LD1 renamed /CPU Tranceiver Driver and Data MUX/LD1
- net LD2 renamed /CPU Tranceiver Driver and Data MUX/LD2
- net LD3 renamed /CPU Tranceiver Driver and Data MUX/LD3
- net LD4 renamed /CPU Tranceiver Driver and Data MUX/LD4
- net LD5 renamed /CPU Tranceiver Driver and Data MUX/LD5
- net LD6 renamed /CPU Tranceiver Driver and Data MUX/LD6
- net LD7 renamed /CPU Tranceiver Driver and Data MUX/LD7
